File: plain60-flex-edition.kicad_pcb (KiCad board)
At the start: 2 copper layers, 284.7 x 94.2 mm, 175 parts, among them J1 HRO-TYPE-C-31-M-12, J2 ISP, J3 ai03_ud, K1 KEYSW, K10 KEYSW, K11 KEYSW, K12 KEYSW, K13 KEYSW, K14 KEYSW, K15 KEYSW, K15-1 KEYSW, K16 KEYSW, K17 KEYSW, K18 KEYSW, K19 KEYSW, K2 KEYSW, K20 KEYSW, K21 KEYSW, K22 KEYSW, K23 KEYSW, K24 KEYSW, K25 KEYSW, K26 KEYSW, K27 KEYSW, K28 KEYSW, K29 KEYSW, K3 KEYSW, K31 KEYSW, K31-1 KEYSW, K32 KEYSW, K33 KEYSW, K34 KEYSW, K35 KEYSW, K36 KEYSW, K37 KEYSW, K38 KEYSW, K39 KEYSW, K4 KEYSW, K40 KEYSW, K41 KEYSW, K42 KEYSW, K43 KEYSW, K44 KEYSW, K44-1 KEYSW, K46 KEYSW, K46-1 KEYSW, K47 KEYSW, K48 KEYSW, K49 KEYSW, K5 KEYSW, K50 KEYSW, K51 KEYSW, K52 KEYSW, K53 KEYSW, K54 KEYSW, K55 KEYSW, K56 KEYSW, K57 KEYSW, K58 KEYSW, K58-1 KEYSW, K59 KEYSW, K6 KEYSW, K61 KEYSW, K61-1 KEYSW, K62 KEYSW, K62-1 KEYSW, K63 KEYSW, K63-1 KEYSW, K67 KEYSW, K67-1 KEYSW, K7 KEYSW, K71 KEYSW, K72 KEYSW, K72-1 KEYSW, K73 KEYSW, K73-1 KEYSW, K74 KEYSW, K74-1 KEYSW, K8 KEYSW, K9 KEYSW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

Commit message: Delete conflicting traces
Routing:
- net Net-(D74-Pad2): track 39.0 -> 9.10 mm
- net Net-(D61-Pad2): track 33.5 -> 6.58 mm
- net col14: track 313.1 -> 290.0 mm
- net row4: track 267.8 -> 247.5 mm
- net Net-(D15-Pad2): track 29.4 -> 9.71 mm
- net Net-(D46-Pad2): track 28.7 -> 10.6 mm
- net GND: track 245.5 -> 228.1 mm
- net col0: track 128.6 -> 112.6 mm
- net Net-(D67-Pad2): track 19.2 -> 7.30 mm
- net RST: track 56.9 -> 45.1 mm
- net Net-(D31-Pad2): track 49.3 -> 39.0 mm, vias 2 -> 1
- net Net-(D1-Pad2): track 27.6 -> 17.7 mm

Commit message: Change footprints to MX+ALPS
Parts:
- K1, K10, K11, K12, K13, K14, K15-1, K17, K18, K19, K2, K20, K21, K22, K23, K24, K25, K26, K27, K28, K3, K32, K33, K34, K35, K36, K37, K38, K39, K4, K40, K41, K42, K47, K48, K49, K5, K50, K51, K52, K53, K54, K55, K56, K57, K59, K6, K62-1, K7, K73-1, K8, K9: footprint Keeb_switches:CHERRY_PLATE_100H -> MX_Alps_Hybrid:MX-1U-NoLED
- K15: footprint Keeb_switches:CHERRY_PCB_200H -> MX_Alps_Hybrid:MX-2U-NoLED
- K16, K29, K61-1, K63-1, K72-1, K74-1: footprint Keeb_switches:CHERRY_PLATE_150H -> MX_Alps_Hybrid:MX-1.5U-NoLED
- K31, K58-1: footprint Keeb_switches:CHERRY_PLATE_175H -> MX_Alps_Hybrid:MX-1.75U-NoLED
- K31-1, K46-1, K61, K62, K63, K71, K72, K73, K74: footprint Keeb_switches:CHERRY_PLATE_125H -> MX_Alps_Hybrid:MX-1.25U-NoLED
- K43: footprint Keeb_switches:CHERRY_PLATE_100H -> MX_Alps_Hybrid:MX-1.5U-NoLED
- K44: footprint Keeb_switches:CHERRY_PCB_225H_F -> MX_Alps_Hybrid:MX-2.25U-NoLED
- K44-1: footprint Keeb_switches:CHERRY_PCB_200H_V -> MX_Alps_Hybrid:MX-ISO-FLIPPED-ReversedStabilizers
- K46: footprint Keeb_switches:CHERRY_PCB_225H -> MX_Alps_Hybrid:MX-2.25U-NoLED
- K58: footprint Keeb_switches:CHERRY_PCB_275H -> MX_Alps_Hybrid:MX-2.75U-NoLED
- K67: footprint Keeb_switches:CHERRY_PCB_625H_F -> MX_Alps_Hybrid:MX-6.25U-ReversedStabilizers-NoLED
- K67-1: footprint Keeb_switches:CHERRY_PCB_700H_F -> MX_Alps_Hybrid:MX-7U-ReversedStabilizers-NoLED
- moved D14 3.57 mm to (245.9, 10.7)
- moved D15 3.57 mm to (249.4, 10.7)
- moved SW1 3.00 mm to (19.1, 57.2)
Connections:
- D46 pad 2: Net-(D46-Pad2) -> Net-(K46-Pad2)
- D59 pad 2: Net-(D59-Pad2) -> Net-(K59-Pad1)
- D61 pad 2: Net-(D61-Pad2) -> Net-(K61-1-Pad2)
- J1 pad 3: (no net) -> unconnected-(J1-Pad3)
- J1 pad 9: (no net) -> unconnected-(J1-Pad9)
- K1 pad 1: Net-(D1-Pad2) -> col0
- K1 pad 2: col0 -> Net-(D1-Pad2)
- K10 pad 1: col9 -> Net-(D10-Pad2)
- K10 pad 2: Net-(D10-Pad2) -> col9
- K11 pad 1: col10 -> Net-(D11-Pad2)
- K11 pad 2: Net-(D11-Pad2) -> col10
- K12 pad 1: col11 -> Net-(D12-Pad2)
- K12 pad 2: Net-(D12-Pad2) -> col11
- K13 pad 1: col12 -> Net-(D13-Pad2)
- K13 pad 2: Net-(D13-Pad2) -> col12
- K14 pad 1: col13 -> Net-(D14-Pad2)
- K14 pad 2: Net-(D14-Pad2) -> col13
- K15 pad 1: col14 -> Net-(D15-Pad2)
- K15 pad 2: Net-(D15-Pad2) -> col14
- K15-1 pad 1: col14 -> Net-(D15-Pad2)
- K15-1 pad 2: Net-(D15-Pad2) -> col14
- K16 pad 1: col0 -> Net-(D16-Pad2)
- K16 pad 2: Net-(D16-Pad2) -> col0
- K17 pad 1: Net-(D17-Pad2) -> col1
- K17 pad 2: col1 -> Net-(D17-Pad2)
- K18 pad 1: col2 -> Net-(D18-Pad2)
- K18 pad 2: Net-(D18-Pad2) -> col2
- K19 pad 1: col3 -> Net-(D19-Pad2)
- K19 pad 2: Net-(D19-Pad2) -> col3
- K2 pad 1: Net-(D2-Pad2) -> col1
- K2 pad 2: col1 -> Net-(D2-Pad2)
- K20 pad 1: col4 -> Net-(D20-Pad2)
- K20 pad 2: Net-(D20-Pad2) -> col4
- K21 pad 1: col5 -> Net-(D21-Pad2)
- K21 pad 2: Net-(D21-Pad2) -> col5
- K22 pad 1: col6 -> Net-(D22-Pad2)
- K22 pad 2: Net-(D22-Pad2) -> col6
- K23 pad 1: col7 -> Net-(D23-Pad2)
- K23 pad 2: Net-(D23-Pad2) -> unconnected-(K23-Pad2)
- K24 pad 1: col8 -> Net-(D24-Pad2)
- K24 pad 2: Net-(D24-Pad2) -> col8
- K25 pad 1: col9 -> Net-(D25-Pad2)
- K25 pad 2: Net-(D25-Pad2) -> col9
- K26 pad 1: col10 -> Net-(D26-Pad2)
- K26 pad 2: Net-(D26-Pad2) -> col10
- K27 pad 1: col11 -> Net-(D27-Pad2)
- K27 pad 2: Net-(D27-Pad2) -> col11
- K28 pad 1: col12 -> Net-(D28-Pad2)
- K28 pad 2: Net-(D28-Pad2) -> col12
- K29 pad 1: col13 -> Net-(D29-Pad2)
- K29 pad 2: Net-(D29-Pad2) -> col13
- K3 pad 1: Net-(D3-Pad2) -> col2
- K3 pad 2: col2 -> Net-(D3-Pad2)
- K31 pad 1: Net-(D31-Pad2) -> unconnected-(K31-Pad1)
- K31 pad 2: col0 -> Net-(D31-Pad2)
- K31-1 pad 1: Net-(D31-Pad2) -> col0
- K31-1 pad 2: col0 -> Net-(D31-Pad2)
- K32 pad 1: Net-(D32-Pad2) -> col1
- K32 pad 2: col1 -> Net-(D32-Pad2)
- K33 pad 1: Net-(D33-Pad2) -> col2
- K33 pad 2: col2 -> Net-(D33-Pad2)
- K34 pad 1: col3 -> Net-(D34-Pad2)
- K34 pad 2: Net-(D34-Pad2) -> col3
- K35 pad 1: col4 -> Net-(D35-Pad2)
- K35 pad 2: Net-(D35-Pad2) -> col4
- K36 pad 1: col5 -> Net-(D36-Pad2)
- K36 pad 2: Net-(D36-Pad2) -> col5
- K37 pad 1: Net-(D37-Pad2) -> col6
- K37 pad 2: col6 -> Net-(D37-Pad2)
- K38 pad 1: col7 -> Net-(D38-Pad2)
- K38 pad 2: Net-(D38-Pad2) -> col7
- K39 pad 1: col8 -> Net-(D39-Pad2)
- K39 pad 2: Net-(D39-Pad2) -> col8
- K4 pad 1: col3 -> Net-(D4-Pad2)
- K4 pad 2: Net-(D4-Pad2) -> col3
- K40 pad 1: col9 -> Net-(D40-Pad2)
- K40 pad 2: Net-(D40-Pad2) -> col9
- K41 pad 1: col10 -> Net-(D41-Pad2)
- K41 pad 2: Net-(D41-Pad2) -> col10
- K42 pad 1: col11 -> Net-(D42-Pad2)
- K42 pad 2: Net-(D42-Pad2) -> col11
- K43 pad 1: col12 -> Net-(D43-Pad2)
- K43 pad 2: Net-(D43-Pad2) -> col12
- K44 pad 1: Net-(D44-Pad2) -> col13
- K44 pad 2: col13 -> Net-(D44-Pad2)
- K46 pad 1: Net-(D46-Pad2) -> col0
- K46 pad 2: col0 -> Net-(K46-Pad2)
- K46-1 pad 1: Net-(D46-Pad2) -> col0
- K46-1 pad 2: col0 -> Net-(K46-Pad2)
- K47 pad 1: Net-(D47-Pad2) -> col1
- K47 pad 2: col1 -> Net-(D47-Pad2)
- K48 pad 1: Net-(D48-Pad2) -> col2
- K48 pad 2: col2 -> Net-(D48-Pad2)
- K49 pad 1: col3 -> Net-(D49-Pad2)
- K49 pad 2: Net-(D49-Pad2) -> col3
- K5 pad 1: col4 -> Net-(D5-Pad2)
- K5 pad 2: Net-(D5-Pad2) -> col4
- K50 pad 1: col4 -> Net-(D50-Pad2)
- K50 pad 2: Net-(D50-Pad2) -> col4
- K51 pad 1: col5 -> Net-(D51-Pad2)
- K51 pad 2: Net-(D51-Pad2) -> col5
- K52 pad 1: col6 -> Net-(D52-Pad2)
- K52 pad 2: Net-(D52-Pad2) -> col6
- K53 pad 1: col7 -> Net-(D53-Pad2)
- K53 pad 2: Net-(D53-Pad2) -> col7
- K54 pad 1: col8 -> Net-(D54-Pad2)
- K54 pad 2: Net-(D54-Pad2) -> col8
- K55 pad 1: col9 -> Net-(D55-Pad2)
- K55 pad 2: Net-(D55-Pad2) -> col9
- K56 pad 1: col10 -> Net-(D56-Pad2)
- K56 pad 2: Net-(D56-Pad2) -> col10
- K57 pad 1: col11 -> Net-(D57-Pad2)
- K57 pad 2: Net-(D57-Pad2) -> col11
- K58 pad 1: col12 -> Net-(D58-Pad2)
- K58 pad 2: Net-(D58-Pad2) -> col12
- K58-1 pad 1: col12 -> Net-(D58-Pad2)
- K58-1 pad 2: Net-(D58-Pad2) -> col12
- K59 pad 1: col13 -> Net-(K59-Pad1)
- K59 pad 2: Net-(D59-Pad2) -> col13
- K6 pad 1: col5 -> Net-(D6-Pad2)
- K6 pad 2: Net-(D6-Pad2) -> col5
- K61 pad 1: Net-(D61-Pad2) -> col0
- K61 pad 2: col0 -> Net-(K61-1-Pad2)
- K61-1 pad 1: Net-(D61-Pad2) -> col0
- K61-1 pad 2: col0 -> Net-(K61-1-Pad2)
- K62 pad 1: Net-(D62-Pad2) -> col1
- K62 pad 2: col1 -> Net-(D62-Pad2)
- K62-1 pad 1: Net-(D62-Pad2) -> col1
- K62-1 pad 2: col1 -> Net-(D62-Pad2)
- K63 pad 1: Net-(D63-Pad2) -> col2
- K63 pad 2: col2 -> Net-(D63-Pad2)
- K63-1 pad 1: Net-(D63-Pad2) -> col2
- K63-1 pad 2: col2 -> Net-(D63-Pad2)
- K67 pad 1: Net-(D67-Pad2) -> col6
- K67 pad 2: col6 -> Net-(D67-Pad2)
- K67-1 pad 1: Net-(D67-Pad2) -> col6
- K67-1 pad 2: col6 -> Net-(D67-Pad2)
- K7 pad 1: col6 -> Net-(D7-Pad2)
- K7 pad 2: Net-(D7-Pad2) -> col6
- K71 pad 1: Net-(D71-Pad2) -> col10
- K71 pad 2: col10 -> Net-(D71-Pad2)
- K72 pad 1: col11 -> Net-(D72-Pad2)
- K72 pad 2: Net-(D72-Pad2) -> col11
- K72-1 pad 1: col11 -> Net-(D72-Pad2)
- K72-1 pad 2: Net-(D72-Pad2) -> col11
- K73 pad 1: col12 -> Net-(D73-Pad2)
- K73 pad 2: Net-(D73-Pad2) -> col12
- K73-1 pad 1: col12 -> Net-(D73-Pad2)
- K73-1 pad 2: Net-(D73-Pad2) -> col12
- K74 pad 1: col13 -> Net-(D74-Pad2)
- K74 pad 2: Net-(D74-Pad2) -> col13
- K74-1 pad 1: col13 -> Net-(D74-Pad2)
- K74-1 pad 2: Net-(D74-Pad2) -> col13
- K8 pad 1: col7 -> Net-(D8-Pad2)
- K8 pad 2: Net-(D8-Pad2) -> col7
- K9 pad 1: col8 -> Net-(D9-Pad2)
- K9 pad 2: Net-(D9-Pad2) -> col8
- U1 pad 42: (no net) -> unconnected-(U1-Pad42)
Routing:
- net Net-(K46-Pad2): track 0.00 -> 31.4 mm
- net Net-(D74-Pad2): track 9.10 -> 38.0 mm
- net col14: track 290.0 -> 315.1 mm
- net row4: track 247.5 -> 267.8 mm
- net GND: track 228.1 -> 245.3 mm
- net RST: track 45.1 -> 60.9 mm
- net Net-(D15-Pad2): track 9.71 -> 25.1 mm
- net col13: track 355.6 -> 369.7 mm
- net col0: track 112.6 -> 125.8 mm
- net Net-(D67-Pad2): track 7.30 -> 19.5 mm
- net Net-(D31-Pad2): track 39.0 -> 50.6 mm
- net Net-(D46-Pad2): track 10.6 -> 0.00 mm
- net Net-(D1-Pad2): track 17.7 -> 28.3 mm
- net Net-(K61-1-Pad2): track 0.00 -> 6.58 mm
- net Net-(D61-Pad2): track 6.58 -> 0.00 mm
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
Commit message: Add AEK support
Parts:
- added K31-2: KEYSW, Alps_Only:ALPS-1.5U, F.Cu at (14.3, 47.6)
- added K62-2: KEYSW, Alps_Only:ALPS-1.25U, F.Cu at (40.5, 85.7)
- added K63-2: KEYSW, Alps_Only:ALPS-1.5U, F.Cu at (66.7, 85.7)
- added K72-2: KEYSW, Alps_Only:ALPS-1.5U, F.Cu at (219.1, 85.7)
- added K73-2: KEYSW, Alps_Only:ALPS-1.25U, F.Cu at (245.3, 85.7)
- moved D61 5.75 mm to (51.6, 86.9)
- moved D62 3.37 mm to (48.4, 86.9)
- moved D72 2.58 mm to (213.5, 86.9)
- moved D63 2.58 mm to (72.2, 86.9)
Connections:
- K31 pad 1: unconnected-(K31-Pad1) -> Net-(D31-Pad2)
- K31 pad 2: Net-(D31-Pad2) -> col0
Routing:
- net Net-(K61-1-Pad2): track 6.58 -> 40.9 mm
- net col11: track 333.4 -> 352.6 mm
- net col12: track 333.9 -> 350.6 mm
- net col2: track 134.5 -> 148.2 mm
- net Net-(D63-Pad2): track 9.68 -> 22.5 mm
- net Net-(D72-Pad2): track 4.98 -> 16.3 mm
- net col1: track 98.6 -> 109.9 mm
- net col0: track 125.8 -> 135.3 mm
- net Net-(D73-Pad2): track 4.98 -> 14.0 mm
- net Net-(D31-Pad2): track 50.6 -> 59.2 mm
- net Net-(D62-Pad2): track 15.6 -> 22.7 mm
- net RST: track 60.9 -> 61.7 mm
Other:
- board text added: "Plain60 MX+ALPS Flex Edition"
- board text removed: "Plain60 Flex Edition"
